File: src/AQ_sensor_SIGFOX.brd (EAGLE design)
At the start: 110 x 64 mm, 35 parts, among them J1 F-1X03-SIP-100-32, SW1 PCM12SMTR, SW2 PCM12SMTR, U3 TEXAS_INSTRUMENTS_LM1117IMP-3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, X1 53048-08

Commit message: sorted DRC
Parts:
- X3: value (none) -> 50ohms
Connections:
- net WISON_RST renamed WISOL_RST
- net GND: now also U$1.22
Routing:
- net +3V3: track 199.8 -> 199.1 mm
- net +5V: track 156.6 -> 156.1 mm
- net DHT_OUT: track 25.8 -> 25.3 mm
Changed lines of the file:
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@@
 </layers>
 <board>
-<fusionteam huburn="a.YnVzaW5lc3M6Y29kZWZvcmFmcmljYTE" projecturn="a.YnVzaW5lc3M6Y29kZWZvcmFmcmljYTEjMjAyMDAzMTgyNzU5ODExNzY" folderUrn="urn:adsk.wipprod:fs.folder:co.JvkIyPCGSUOTXoHwebdYWw" urn="urn:adsk.wipprod:dm.lineage:Uf6rQSBaT3aBi3ddeRhs7w"  versionUrn="urn:adsk.wipprod:fs.file:vf.Uf6rQSBaT3aBi3ddeRhs7w?version=5" camFileUrn="" camFileVersionUrn="" lastpublishedchangeguid="a7db0acd-e38e-caf0-5e21-a538b23dd096"/>
+<fusionsync huburn="a.YnVzaW5lc3M6Y29kZWZvcmFmcmljYTE" projecturn="a.YnVzaW5lc3M6Y29kZWZvcmFmcmljYTEjMjAyMTEwMDU0NTIxNjk1MjY" f3durn="urn:adsk.wipprod:dm.lineage:PAO7QyUTTHaXe7WWxUpZLw" pcbguid="" lastpulledtime="" lastsyncedchangeguid="" latestrevisionid="57a06fd7-7e1d-427a-903e-aaa3c097e9e6" lastsyncedrevisionid="57a06fd7-7e1d-427a-903e-aaa3c097e9e6" lastboardhashguid="d1a07737-3213-db7d-5466-6e395773a376" lastpushedtime="2021-10-05T09:37:29Z" linktopcb3d="true"/>
+<fusionteam huburn="a.YnVzaW5lc3M6Y29kZWZvcmFmcmljYTE" projecturn="a.YnVzaW5lc3M6Y29kZWZvcmFmcmljYTEjMjAyMTEwMDU0NTIxNjk1MjY" folderUrn="urn:adsk.wipprod:fs.folder:co.dgCpAfyER96Zuqcgu0tqyw" urn="urn:adsk.wipprod:dm.lineage:YCYfI4sjTE6TtrKYoMCkVA"  versionUrn="urn:adsk.wipprod:fs.file:vf.YCYfI4sjTE6TtrKYoMCkVA?version=1" camFileUrn="" camFileVersionUrn="" lastpublishedchangeguid="419bff36-aa4a-df2b-38c0-ff70da88a0eb"/>
 <plain>
 <wire x1="0" y1="0" x2="110" y2="0" width="0" layer="20"/>
@@
 <attribute name="VALUE" x="98.715" y="56.15" size="1.27" layer="27" rot="R90"/>
 </element>
-<element name="J1" library="AQ_sensor_GSM" library_urn="urn:adsk.eagle:library:30300195" package="SIP-100-03-32" package3d_urn="urn:adsk.eagle:package:30300264/2" value="F-1X03-SIP-100-32" x="107.3" y="49.15" smashed="yes" rot="R270">
+<element name="J1" library="AQ_sensor_GSM" library_urn="urn:adsk.eagle:library:30300195" package="SIP-100-03-32" package3d_urn="urn:adsk.eagle:package:30300264/3" value="F-1X03-SIP-100-32" x="107.3" y="49.15" smashed="yes" rot="R270">
 <attribute name="NAME" x="106.03" y="53.595" size="1.016" layer="25" ratio="18"/>
 <attribute name="VALUE" x="109.63" y="45.37" size="0.8128" layer="27" ratio="10" rot="R90"/>
@@
 <attribute name="VALUE" x="24.005" y="6.265" size="1.27" layer="27" rot="R90"/>
 </element>
-<element name="X3" library="AQ_sensor_GSM" library_urn="urn:adsk.eagle:library:30260301" package="SMA_EDGELAUNCH_UFL" package3d_urn="urn:adsk.eagle:package:30260396/1" value="" x="26.8" y="0.5" smashed="yes" rot="R90">
+<element name="X3" library="AQ_sensor_GSM" library_urn="urn:adsk.eagle:library:30260301" package="SMA_EDGELAUNCH_UFL" package3d_urn="urn:adsk.eagle:package:30260396/1" value="50ohms" x="26.8" y="0.5" smashed="yes" rot="R90">
 <attribute name="NAME" x="20.015" y="3.08" size="1.016" layer="25" ratio="18" rot="R270"/>
 <attribute name="VALUE" x="34.42" y="5.58" size="0.8128" layer="27" ratio="10" rot="R270"/>
@@
 <contactref element="U$1" pad="31"/>
 <contactref element="U$1" pad="28"/>
+<contactref element="U$1" pad="22"/>
 </signal>
 <signal name="+5V" class="1">
@@
 <contactref element="U3" pad="3"/>
 <contactref element="SW1" pad="1"/>
-<wire x1="102.51" y1="14.18" x2="102.76" y2="14.43" width="0.4" layer="1"/>
-<wire x1="89.775" y1="35.2" x2="89.805" y2="35.17" width="0.4" layer="16"/>
 <wire x1="85.45" y1="3.75" x2="85.45" y2="5.65" width="0.6" layer="1"/>
-<wire x1="85.5" y1="5.7" x2="85.45" y2="5.65" width="0.6" layer="1"/>
 <wire x1="85.45" y1="5.65" x2="85.45" y2="8.95" width="1.2" layer="1"/>
 <wire x1="95.5" y1="10.9" x2="97.9" y2="13.3" width="1.2" layer="1"/>
@@
 <wire x1="102" y1="35.3" x2="100.3" y2="35.3" width="1.2" layer="1"/>
 <wire x1="99.18" y1="35.25" x2="99.18" y2="36.48" width="0.6" layer="1"/>
-<wire x1="99.18" y1="36.48" x2="99.2" y2="36.5" width="0.6" layer="1"/>
 <wire x1="89.805" y1="35.17" x2="88.13" y2="35.17" width="0.6" layer="16"/>
-<wire x1="88.13" y1="35.17" x2="88.1" y2="35.2" width="0.6" layer="16"/>
 <wire x1="88.13" y1="35.17" x2="83.93" y2="35.17" width="1.2" layer="16"/>
 <wire x1="83.93" y1="35.17" x2="83.9" y2="35.2" width="1.2" layer="16"/>
@@
 <wire x1="69.2" y1="57.1" x2="76" y2="57.1" width="1.2" layer="16"/>
 <wire x1="86.715" y1="59.15" x2="86.715" y2="57.515" width="0.6" layer="16"/>
-<wire x1="86.715" y1="57.515" x2="86.7" y2="57.5" width="0.6" layer="16"/>
 <wire x1="86.715" y1="56.815" x2="86.715" y2="57.515" width="1.2" layer="16"/>
 <wire x1="76" y1="57.1" x2="77.1" y2="56" width="1.2" layer="16"/>
@@
 <contactref element="U3" pad="4"/>
 <contactref element="C8" pad="1"/>
-<wire x1="85.52" y1="32.98" x2="85.8" y2="32.98" width="0.4" layer="16"/>
-<wire x1="89.695" y1="32.98" x2="89.805" y2="32.87" width="0.4" layer="16"/>
 <wire x1="95.955" y1="32.87" x2="91.63" y2="32.87" width="1.2" layer="16"/>
-<wire x1="91.63" y1="32.87" x2="91.6" y2="32.9" width="1.2" layer="16"/>
 <wire x1="91.63" y1="32.87" x2="89.805" y2="32.87" width="0.6" layer="16"/>
-<wire x1="89.805" y1="32.87" x2="88.53" y2="32.87" width="0.6" layer="16"/>
-<wire x1="88.53" y1="32.87" x2="88.5" y2="32.9" width="0.6" layer="16"/>
-<wire x1="88.53" y1="32.87" x2="87.03" y2="32.87" width="1.2" layer="16"/>
-<wire x1="87.03" y1="32.87" x2="87" y2="32.9" width="1.2" layer="16"/>
-<wire x1="87.03" y1="32.87" x2="85.63" y2="32.87" width="0.6" layer="16"/>
+<wire x1="85.63" y1="32.87" x2="87.03" y2="32.87" width="0.6" layer="16"/>
 <wire x1="85.63" y1="32.87" x2="85.52" y2="32.98" width="0.6" layer="16"/>
 <wire x1="85.52" y1="32.98" x2="83.82" y2="32.98" width="0.6" layer="16"/>
-<wire x1="83.82" y1="32.98" x2="83.8" y2="33" width="0.6" layer="16"/>
 <wire x1="83.82" y1="32.98" x2="82.18" y2="32.98" width="1.2" layer="16"/>
 <wire x1="82.18" y1="32.98" x2="80.7" y2="31.5" width="1.2" layer="16"/>
@@
 <wire x1="17.3" y1="35.1" x2="9" y2="26.8" width="1.2" layer="16"/>
 <wire x1="9" y1="26.8" x2="9" y2="13.6" width="1.2" layer="16"/>
-<wire x1="16.75" y1="12" x2="16.8" y2="12.05" width="0.6" layer="1"/>
 <wire x1="16.85" y1="14.2" x2="16.85" y2="12.1" width="0.6" layer="1"/>
 <wire x1="16.85" y1="12.1" x2="16.8" y2="12.05" width="0.6" layer="1"/>
@@
 <wire x1="17.6782" y1="6.2782" x2="21.1" y2="9.7" width="1.2" layer="1"/>
 <contactref element="R5" pad="1"/>
-<wire x1="103.03" y1="46.59" x2="103.04" y2="46.6" width="0.6" layer="1"/>
 <contactref element="J1" pad="3"/>
 <wire x1="97.78" y1="44.94" x2="97.78" y2="46.08" width="1.2" layer="1"/>
@@
 <wire x1="103.02" y1="46.6" x2="103.03" y2="46.59" width="0.6" layer="1"/>
 <wire x1="103.03" y1="46.59" x2="104.29" y2="46.59" width="0.6" layer="1"/>
-<wire x1="104.29" y1="46.59" x2="104.3" y2="46.6" width="0.6" layer="1"/>
 <wire x1="104.29" y1="46.59" x2="107.28" y2="46.59" width="1.2" layer="1"/>
 <wire x1="107.28" y1="46.59" x2="107.3" y2="46.61" width="1.2" layer="1"/>
@@
 <wire x1="7.1" y1="8.8" x2="9.4" y2="8.8" width="1.2" layer="1"/>
 <wire x1="9.4" y1="8.8" x2="10.55" y2="8.8" width="0.6" layer="1"/>
+<wire x1="87.03" y1="32.87" x2="88.17" y2="32.87" width="1.2" layer="16"/>
+<wire x1="88.17" y1="32.87" x2="89.805" y2="32.87" width="0.6" layer="16"/>
 </signal>
 <signal name="DHT_OUT">
@@
 <contactref element="R5" pad="2"/>
 <contactref element="SV1" pad="6"/>
-<wire x1="102.82" y1="48.5" x2="103.03" y2="48.29" width="0.4" layer="1"/>
 <wire x1="85.08" y1="47.18" x2="85.08" y2="44.94" width="0.3" layer="1"/>
-<wire x1="85.08" y1="47.18" x2="86.3" y2="48.4" width="0.3" layer="1"/>
-<wire x1="103.03" y1="48.29" x2="103.14" y2="48.4" width="0.3" layer="1"/>
-<wire x1="86.3" y1="48.4" x2="102.92" y2="48.4" width="0.3" layer="1"/>
-<wire x1="102.92" y1="48.4" x2="103.03" y2="48.29" width="0.3" layer="1"/>
-<wire x1="103.03" y1="48.29" x2="103.24" y2="48.5" width="0.3" layer="1"/>
-<wire x1="105.25" y1="49.15" x2="107.3" y2="49.15" width="0.3" layer="1"/>
-<wire x1="103.24" y1="48.5" x2="104.6" y2="48.5" width="0.3" layer="1"/>
-<wire x1="104.6" y1="48.5" x2="105.25" y2="49.15" width="0.3" layer="1"/>
+<wire x1="107.3" y1="49.15" x2="105.25" y2="49.15" width="0.3" layer="1"/>
+<wire x1="104.39" y1="48.29" x2="103.03" y2="48.29" width="0.3" layer="1"/>
+<wire x1="105.25" y1="49.15" x2="104.39" y2="48.29" width="0.3" layer="1"/>
+<wire x1="103.03" y1="48.29" x2="86.19" y2="48.29" width="0.3" layer="1"/>
+<wire x1="86.19" y1="48.29" x2="85.08" y2="47.18" width="0.3" layer="1"/>
 </signal>
 <signal name="PMS_LED">
@@
 <contactref element="R3" pad="2"/>
 <contactref element="C5" pad="1"/>
-<wire x1="12.45" y1="9" x2="12.45" y2="9.2" width="0.3" layer="1"/>
 <wire x1="14.86" y1="16.82" x2="13.92" y2="16.82" width="0.6" layer="1"/>
 <wire x1="13.6" y1="16.5" x2="13.6" y2="15.9" width="0.6" layer="1"/>
@@
 <wire x1="81.5" y1="49.2" x2="82.54" y2="48.16" width="0.3" layer="1"/>
 </signal>
-<signal name="WISON_RST">
+<signal name="WISOL_RST">
 <contactref element="U$1" pad="13"/>
 </signal>
@@
 <mfgpreviewcolor name="substratecolor" color="0xFF786E46"/>
 </mfgpreviewcolors>
-<errors>
-</errors>
 </board>
 </drawing>
@@
 </note>
 <note version="8.3" severity="warning">
+Since Version 8.3, EAGLE supports Fusion synchronisation.
+This feature will not be available in this version and saving
+the document will break the link to the Fusion PCB feature.
+</note>
+<note version="8.3" severity="warning">
