File: src/AQ_sensor_SIGFOX.sch (EAGLE design)
At the start: 35 parts, among them J1 F-1X03-SIP-100-32, SW1 PCM12SMTR, SW2 PCM12SMTR, U3 TEXAS_INSTRUMENTS_LM1117IMP-3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, X1 53048-08

Commit message: sorted DRC
Parts:
- X3: value (none) -> 50ohms
Connections:
- net WISON_RST renamed WISOL_RST
- net GND: now also U$1.22
Changed lines of the file:
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@@
 <setting verticaltext="up"/>
 </settings>
-<grid distance="0.01" unitdist="inch" unit="inch" style="dots" multiple="1" display="yes" altdistance="0.01" altunitdist="inch" altunit="inch"/>
+<grid distance="0.1" unitdist="inch" unit="inch" style="lines" multiple="1" display="no" altdistance="0.01" altunitdist="inch" altunit="inch"/>
 <layers>
 <layer number="1" name="Top" color="4" fill="1" visible="no" active="no"/>
@@
 </layers>
 <schematic xreflabel="%F%N/%S.%C%R" xrefpart="/%S.%C%R">
-<fusionteam huburn="a.YnVzaW5lc3M6Y29kZWZvcmFmcmljYTE" projecturn="a.YnVzaW5lc3M6Y29kZWZvcmFmcmljYTEjMjAyMDAzMTgyNzU5ODExNzY" folderUrn="urn:adsk.wipprod:fs.folder:co.JvkIyPCGSUOTXoHwebdYWw" urn="urn:adsk.wipprod:dm.lineage:lKNtYnu6R0Wf073pCdF1XA"  versionUrn="urn:adsk.wipprod:fs.file:vf.lKNtYnu6R0Wf073pCdF1XA?version=5" camFileUrn="" camFileVersionUrn="" lastpublishedchangeguid="f7d3d892-1735-423b-440c-40111b257b6f"/>
+<fusionteam huburn="a.YnVzaW5lc3M6Y29kZWZvcmFmcmljYTE" projecturn="a.YnVzaW5lc3M6Y29kZWZvcmFmcmljYTEjMjAyMTEwMDU0NTIxNjk1MjY" folderUrn="urn:adsk.wipprod:fs.folder:co.dgCpAfyER96Zuqcgu0tqyw" urn="urn:adsk.wipprod:dm.lineage:U0wo6XjgT5K0S-mF1DSGnQ"  versionUrn="urn:adsk.wipprod:fs.file:vf.U0wo6XjgT5K0S-mF1DSGnQ?version=1" camFileUrn="" camFileVersionUrn="" lastpublishedchangeguid="60c72a1a-1266-8ebc-7aaf-a876d39807dd"/>
 <attributes>
 </attributes>
@@
 <part name="GND2" library="supply1" library_urn="urn:adsk.eagle:library:371" deviceset="GND" device=""/>
 <part name="X1" library="AQ_sensor_GSM" library_urn="urn:adsk.eagle:library:30300195" deviceset="53?-08" device="048" package3d_urn="urn:adsk.eagle:package:30300278/2"/>
-<part name="J1" library="AQ_sensor_GSM" library_urn="urn:adsk.eagle:library:30300195" deviceset="F-1X03-" device="SIP-100-32" package3d_urn="urn:adsk.eagle:package:30300264/2"/>
+<part name="J1" library="AQ_sensor_GSM" library_urn="urn:adsk.eagle:library:30300195" deviceset="F-1X03-" device="SIP-100-32" package3d_urn="urn:adsk.eagle:package:30300264/3"/>
 <part name="SV1" library="AQ_sensor_GSM" library_urn="urn:adsk.eagle:library:30300195" deviceset="FE15-1" device="" package3d_urn="urn:adsk.eagle:package:30300273/2"/>
 <part name="SV2" library="AQ_sensor_GSM" library_urn="urn:adsk.eagle:library:30300195" deviceset="FE15-1" device="" package3d_urn="urn:adsk.eagle:package:30300273/2"/>
@@
 <part name="L1" library="OPL_Inductor" deviceset="SMD-INDUCTOR-2.2UH-20%-1.2A(0805)" device="" package3d_urn="urn:adsk.eagle:package:8004743/1" value="47NH"/>
 <part name="R2" library="rcl" library_urn="urn:adsk.eagle:library:334" deviceset="R-EU_" device="R0603" package3d_urn="urn:adsk.eagle:package:23555/3" value="0R"/>
-<part name="X3" library="AQ_sensor_GSM" library_urn="urn:adsk.eagle:library:30260301" deviceset="SMACONNECTOR" device="_EDGE_UFL" package3d_urn="urn:adsk.eagle:package:30260396/1"/>
+<part name="X3" library="AQ_sensor_GSM" library_urn="urn:adsk.eagle:library:30260301" deviceset="SMACONNECTOR" device="_EDGE_UFL" package3d_urn="urn:adsk.eagle:package:30260396/1" value="50ohms"/>
 <part name="GND11" library="supply1" library_urn="urn:adsk.eagle:library:371" deviceset="GND" device=""/>
 <part name="GND16" library="supply1" library_urn="urn:adsk.eagle:library:371" deviceset="GND" device=""/>
@@
 <attribute name="VALUE" x="321.564" y="206.756" size="1.778" layer="96"/>
 </instance>
-<instance part="GND27" gate="1" x="322.834" y="199.39" smashed="yes" rot="R90">
-<attribute name="VALUE" x="325.374" y="196.85" size="1.778" layer="96" rot="R90"/>
+<instance part="GND27" gate="1" x="325.374" y="199.39" smashed="yes" rot="R90">
+<attribute name="VALUE" x="327.914" y="196.85" size="1.778" layer="96" rot="R90"/>
 </instance>
 <instance part="GND28" gate="1" x="321.31" y="191.008" smashed="yes">
@@
 <wire x1="324.104" y1="214.63" x2="320.548" y2="214.63" width="0.1524" layer="91"/>
 </segment>
+<segment>
+<pinref part="U$1" gate="G$1" pin="22"/>
+<pinref part="GND27" gate="1" pin="GND"/>
+<wire x1="320.548" y1="199.39" x2="322.834" y2="199.39" width="0.1524" layer="91"/>
+</segment>
 </net>
 <net name="+5V" class="1">
@@
 </segment>
 </net>
-<net name="WISON_RST" class="0">
+<net name="WISOL_RST" class="0">
 <segment>
 <pinref part="U$1" gate="G$1" pin="GPIO9"/>
